File: Digital Voltmeter/Digital Voltmeter.kicad_pcb (KiCad board)
At the start: 2 copper layers, 70.8 x 61.2 mm, 23 parts, among them U1 L78L05_SO8, U2 ICL7660S, U3 ICL7107, U4 MAN6960, U5 MAN6960, U6 MAN6960, U7 MAN6960

Commit message: before changing some components
Other:
- board size 70.8 x 61.2 mm -> 70.8 x 61.1 mm
Changed lines of the file:
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@@
       (effects (font (size 1 1) (thickness 0.15)))
     )
-    (fp_text value 10u (at 0 -1.778 270) (layer F.Fab)
+    (fp_text value 10u (at 0 -1.778 270) (layer F.SilkS)
       (effects (font (size 1 1) (thickness 0.15)))
     )
@@
     (at 119.126 89.0905)
     (attr smd)
-    (fp_text reference U2 (at 0 -4.7625) (layer F.SilkS)
-      (effects (font (size 1.64393 1.64393) (thickness 0.05)))
-    )
-    (fp_text value ICL7660S (at -0.3175 4.191) (layer F.Fab)
-      (effects (font (size 1.64373 1.64373) (thickness 0.05)))
+    (fp_text reference U2 (at 0 -3.3655) (layer F.SilkS)
+      (effects (font (size 1 1) (thickness 0.15)))
+    )
+    (fp_text value ICL7660S (at 0 3.6195) (layer F.Fab)
+      (effects (font (size 1 1) (thickness 0.15)))
     )
     (fp_arc (start 0 -2.4892) (end -0.3048 -2.4892) (angle -180) (layer F.SilkS) (width 0.1524))
@@
     )
   )
-  (gr_line (start 104 75.6) (end 104 136.8425) (layer Edge.Cuts) (width 0.2))
+  (gr_line (start 104 75.6) (end 104 136.7155) (layer Edge.Cuts) (width 0.2))
   (gr_line (start 174.75 75.6) (end 104 75.6) (layer Edge.Cuts) (width 0.2))
   (gr_line (start 174.75 136.7155) (end 174.75 75.6) (layer Edge.Cuts) (width 0.2))
   (gr_line (start 104 136.7155) (end 174.75 136.7155) (layer Edge.Cuts) (width 0.2))
-  (via (at 132.6515 94.361) (size 0.8) (drill 0.4) (layers F.Cu B.Cu) (net 30))
-  (via (at 137.414 89.662) (size 0.8) (drill 0.4) (layers F.Cu B.Cu) (net 30))
-  (via (at 114.4905 104.013) (size 0.8) (drill 0.4) (layers F.Cu B.Cu) (net 6))
-  (via (at 123.3805 97.409) (size 0.8) (drill 0.4) (layers F.Cu B.Cu) (net 11))
-  (via (at 114.4905 101.2825) (size 0.8) (drill 0.4) (layers F.Cu B.Cu) (net 11))
-  (via (at 117.221 131.5085) (size 0.8) (drill 0.4) (layers F.Cu B.Cu) (net 6))
-  (via (at 114.427 97.409) (size 0.8) (drill 0.4) (layers F.Cu B.Cu) (net 6))
-  (via (at 123.3805 101.2825) (size 0.8) (drill 0.4) (layers F.Cu B.Cu) (net 6))
-  (via (at 119.634 119.38) (size 0.8) (drill 0.4) (layers F.Cu B.Cu) (net 11))
-  (via (at 114.8715 89.7255) (size 0.8) (drill 0.4) (layers F.Cu B.Cu) (net 10))
   (segment (start 129.1995 106.8475) (end 126.492 106.8475) (width 0.25) (layer F.Cu) (net 1))
   (segment (start 130.429 108.077) (end 129.1995 106.8475) (width 0.25) (layer F.Cu) (net 1))
@@
   (segment (start 129.7305 129.0955) (end 130.429 128.397) (width 0.25) (layer F.Cu) (net 5))
   (segment (start 125.6665 129.0955) (end 129.7305 129.0955) (width 0.25) (layer F.Cu) (net 5))
+  (via (at 114.4905 104.013) (size 0.8) (drill 0.4) (layers F.Cu B.Cu) (net 6))
+  (via (at 117.221 131.5085) (size 0.8) (drill 0.4) (layers F.Cu B.Cu) (net 6))
+  (via (at 114.427 97.409) (size 0.8) (drill 0.4) (layers F.Cu B.Cu) (net 6))
+  (via (at 123.3805 101.2825) (size 0.8) (drill 0.4) (layers F.Cu B.Cu) (net 6))
   (segment (start 149.6695 130.937) (end 153.289 127.3175) (width 0.25) (layer B.Cu) (net 6))
   (segment (start 145.669 130.937) (end 149.6695 130.937) (width 0.25) (layer B.Cu) (net 6))
@@
   (segment (start 126.492 96.2035) (end 126.492 98.7445) (width 0.25) (layer F.Cu) (net 9))
   (segment (start 126.492 95.616) (end 126.492 96.2035) (width 0.25) (layer F.Cu) (net 9))
+  (via (at 114.8715 89.7255) (size 0.8) (drill 0.4) (layers F.Cu B.Cu) (net 10))
   (segment (start 109.526 119.3165) (end 108.776 119.3165) (width 0.25) (layer F.Cu) (net 10))
   (segment (start 112.8395 122.63) (end 109.526 119.3165) (width 0.25) (layer F.Cu) (net 10))
@@
   (segment (start 114.750998 99.949) (end 108.776 105.923998) (width 0.25) (layer F.Cu) (net 10))
   (segment (start 116.2355 99.949) (end 114.750998 99.949) (width 0.25) (layer F.Cu) (net 10))
+  (via (at 123.3805 97.409) (size 0.8) (drill 0.4) (layers F.Cu B.Cu) (net 11))
+  (via (at 114.4905 101.2825) (size 0.8) (drill 0.4) (layers F.Cu B.Cu) (net 11))
+  (via (at 119.634 119.38) (size 0.8) (drill 0.4) (layers F.Cu B.Cu) (net 11))
   (segment (start 119.5705 119.3165) (end 119.634 119.38) (width 0.25) (layer F.Cu) (net 11))
   (segment (start 116.776 119.3165) (end 119.5705 119.3165) (width 0.25) (layer F.Cu) (net 11))
@@
   (segment (start 147.224303 98.051501) (end 145.509803 96.337001) (width 0.25) (layer B.Cu) (net 29))
   (segment (start 168.529 104.5845) (end 161.996001 98.051501) (width 0.25) (layer B.Cu) (net 29))
+  (via (at 132.6515 94.361) (size 0.8) (drill 0.4) (layers F.Cu B.Cu) (net 30))
+  (via (at 137.414 89.662) (size 0.8) (drill 0.4) (layers F.Cu B.Cu) (net 30))
   (segment (start 169.050761 79.367499) (end 141.422001 79.367499) (width 0.25) (layer F.Cu) (net 30))
   (segment (start 170.066011 80.382749) (end 169.050761 79.367499) (width 0.25) (layer F.Cu) (net 30))

Commit message: replaced parts
Parts:
- C2, C5: footprint Capacitor_SMD:C_0603_1608Metric -> Capacitor_SMD:C_0603_1608Metric_Pad1.05x0.95mm_HandSolder
- C3, C4, C8: footprint Capacitor_SMD:C_0805_2012Metric -> Capacitor_SMD:C_0603_1608Metric_Pad1.05x0.95mm_HandSolder
- C6, C7, C9: footprint Capacitor_SMD:C_0402_1005Metric -> Capacitor_SMD:C_0603_1608Metric_Pad1.05x0.95mm_HandSolder
- R1: footprint Resistor_SMD:R_0805_2012Metric -> Resistor_SMD:R_0603_1608Metric_Pad1.05x0.95mm_HandSolder
- R2, R4, R5: footprint Resistor_SMD:R_0402_1005Metric -> Resistor_SMD:R_0603_1608Metric_Pad1.05x0.95mm_HandSolder
- R3, R6: footprint Resistor_SMD:R_0201_0603Metric -> Resistor_SMD:R_0603_1608Metric_Pad1.05x0.95mm_HandSolder
- moved C4 1.33 mm to (126.5, 87.8)
- moved C5 0.91 mm to (122.1, 107.2)
- moved C2 0.83 mm to (112.0, 129.5)
- moved R4 0.83 mm to (126.5, 129.5)
- moved R1 0.83 mm to (117.9, 107.2)
- moved R2 0.83 mm to (126.5, 107.2)
- moved R6 0.63 mm to (126.5, 83.5)
- moved R3 0.51 mm to (126.5, 98.6)
- moved R5 0.51 mm to (116.7, 129.5)
- moved C8 0.44 mm to (126.5, 94.2)
- moved C3 0.06 mm to (112.0, 89.5)
Routing:
- net GND: track 67.6 -> 71.0 mm
- net -5V: track 14.6 -> 13.3 mm
- net Net-(R4-Pad1): track 5.05 -> 4.05 mm
- net /Vin-: track 29.5 -> 30.5 mm
- net Net-(R6-Pad1): track 47.3 -> 46.4 mm
- net Net-(C5-Pad2): track 13.3 -> 12.6 mm
- net Net-(R5-Pad2): track 11.0 -> 11.5 mm
- net Net-(C8-Pad1): track 5.81 -> 6.35 mm

Commit message: passing DMC
Parts:
- added G***: LOGO, logos:ieee-logo-inv, F.Cu at (109.5, 80.8)
- added G***: LOGO, logos:bac-logo, F.Cu at (119.3, 80.5)
- added J1: Conn_01x02_Male, Connector_PinHeader_2.54mm:PinHeader_1x02_P2.54mm_Vertical, F.Cu at (112.8, 109.0)
- added J2: Conn_01x02_Male, Connector_PinHeader_2.54mm:PinHeader_1x02_P2.54mm_Vertical, F.Cu at (108.8, 98.0)
Routing:
- net /Vin-: track 30.5 -> 40.6 mm
- net /Vin=9V: track 37.1 -> 45.6 mm, vias 3 -> 5
- net /Vin+: track 0.00 -> 6.21 mm
- net GND: track 71.0 -> 76.6 mm
