File: Digital Voltmeter/Digital Voltmeter.sch (KiCad schematic (older format))
At the start: 23 parts, among them U1 L78L05_SO8, U2 ICL7660S, U3 ICL7107, U4 MAN6960, U5 MAN6960, U6 MAN6960, U7 MAN6960

Commit message: adding footprints
Parts:
- C1: footprint (none) -> Capacitor_SMD:CP_Elec_10x10
- C2, C5: footprint (none) -> Capacitor_SMD:C_0603_1608Metric
- C3, C4, C8: footprint (none) -> Capacitor_SMD:C_0805_2012Metric
- C6, C7, C9: footprint (none) -> Capacitor_SMD:C_0402_1005Metric
- R1: footprint (none) -> Resistor_SMD:R_0805_2012Metric
- R2, R4, R5: footprint (none) -> Resistor_SMD:R_0402_1005Metric
- R3, R6: footprint (none) -> Resistor_SMD:R_0201_0603Metric
- U2: symbol Digital~Voltmeter:ICL7660S -> Digital_Voltmeter:ICL7660S
- U3: symbol Digital~Voltmeter:ICL7107 -> Digital_Voltmeter:ICL7107
- U4, U5, U6, U7: symbol Digital~Voltmeter:MAN6960 -> Digital_Voltmeter:MAN6960
Connections:
- wire segments 91 -> 90
Changed lines of the file:
@@
 F 0 "C2" H 2328 2346 50  0000 L CNN
 F 1 "2.2u" H 2328 2255 50  0000 L CNN
-F 2 "" H 2150 2300 50  0001 C CNN
+F 2 "Capacitor_SMD:C_0603_1608Metric" H 2150 2300 50  0001 C CNN
 F 3 "" H 2150 2300 50  0001 C CNN
 	1    2150 2300
@@
 $EndComp
 $Comp
-L Digital~Voltmeter:ICL7660S U2
+L Digital_Voltmeter:ICL7660S U2
 U 1 1 5BC8ADD6
 P 3400 2300
@@
 F 0 "C3" H 2978 2346 50  0000 L CNN
 F 1 "10u" H 2978 2255 50  0000 L CNN
-F 2 "" H 2800 2300 50  0001 C CNN
+F 2 "Capacitor_SMD:C_0805_2012Metric" H 2800 2300 50  0001 C CNN
 F 3 "" H 2800 2300 50  0001 C CNN
 	1    2800 2300
@@
 F 0 "C4" H 4178 2596 50  0000 L CNN
 F 1 "10u" H 4178 2505 50  0000 L CNN
-F 2 "" H 4000 2550 50  0001 C CNN
+F 2 "Capacitor_SMD:C_0805_2012Metric" H 4000 2550 50  0001 C CNN
 F 3 "" H 4000 2550 50  0001 C CNN
 	1    4000 2550
 	1    0    0    -1
 $EndComp
-Wire Wire Line
-	2150 1900 3400 1900
 Wire Wire Line
 	3050 2050 2800 2050
@@
 F 0 "C1" H 1728 2346 50  0000 L CNN
 F 1 "470u" H 1728 2255 50  0000 L CNN
-F 2 "" H 1550 2300 50  0001 C CNN
+F 2 "Capacitor_SMD:CP_Elec_10x10" H 1550 2300 50  0001 C CNN
 F 3 "" H 1550 2300 50  0001 C CNN
 	1    1550 2300
@@
 F 0 "C6" H 6028 4996 50  0000 L CNN
 F 1 "100nF" H 6028 4905 50  0000 L CNN
-F 2 "" H 5850 4950 50  0001 C CNN
+F 2 "Capacitor_SMD:C_0402_1005Metric" H 5850 4950 50  0001 C CNN
 F 3 "" H 5850 4950 50  0001 C CNN
 	1    5850 4950
@@
 F 0 "C5" H 6028 3696 50  0000 L CNN
 F 1 "10nF" H 6028 3605 50  0000 L CNN
-F 2 "" H 5850 3650 50  0001 C CNN
+F 2 "Capacitor_SMD:C_0603_1608Metric" H 5850 3650 50  0001 C CNN
 F 3 "" H 5850 3650 50  0001 C CNN
 	1    5850 3650
@@
 F 0 "C9" V 6000 5300 50  0000 C CNN
 F 1 "100pF" V 6000 5600 50  0000 C CNN
-F 2 "" H 6100 5400 50  0001 C CNN
+F 2 "Capacitor_SMD:C_0402_1005Metric" H 6100 5400 50  0001 C CNN
 F 3 "" H 6100 5400 50  0001 C CNN
 	1    6100 5400
@@
 F 0 "C8" V 6150 4400 50  0000 C CNN
 F 1 "220nF" V 6150 4700 50  0000 C CNN
-F 2 "" H 6100 4500 50  0001 C CNN
+F 2 "Capacitor_SMD:C_0805_2012Metric" H 6100 4500 50  0001 C CNN
 F 3 "" H 6100 4500 50  0001 C CNN
 	1    6100 4500
@@
 F 0 "C7" V 6150 4000 50  0000 C CNN
 F 1 "47nF" V 6150 4250 50  0000 C CNN
-F 2 "" H 6100 4100 50  0001 C CNN
+F 2 "Capacitor_SMD:C_0402_1005Metric" H 6100 4100 50  0001 C CNN
 F 3 "" H 6100 4100 50  0001 C CNN
 	1    6100 4100
@@
 F 0 "R4" V 6150 5450 50  0000 C CNN
 F 1 "180k" V 6150 5800 50  0000 C CNN
-F 2 "" V 6030 5600 50  0001 C CNN
+F 2 "Resistor_SMD:R_0402_1005Metric" V 6030 5600 50  0001 C CNN
 F 3 "~" H 6100 5600 50  0001 C CNN
 	1    6100 5600
@@
 F 0 "R3" V 6150 4150 50  0000 C CNN
 F 1 "470k" V 6150 4500 50  0000 C CNN
-F 2 "" V 6030 4300 50  0001 C CNN
+F 2 "Resistor_SMD:R_0201_0603Metric" V 6030 4300 50  0001 C CNN
 F 3 "~" H 6100 4300 50  0001 C CNN
 	1    6100 4300
@@
 F 0 "R2" H 5570 3696 50  0000 L CNN
 F 1 "12k" H 5570 3605 50  0000 L CNN
-F 2 "" V 5430 3650 50  0001 C CNN
+F 2 "Resistor_SMD:R_0402_1005Metric" V 5430 3650 50  0001 C CNN
 F 3 "~" H 5500 3650 50  0001 C CNN
 	1    5500 3650
@@
 F 0 "R1" V 4943 3900 50  0000 C CNN
 F 1 "1M" V 5034 3900 50  0000 C CNN
-F 2 "" V 5080 3900 50  0001 C CNN
+F 2 "Resistor_SMD:R_0805_2012Metric" V 5080 3900 50  0001 C CNN
 F 3 "~" H 5150 3900 50  0001 C CNN
 	1    5150 3900
@@
 F 0 "R5" V 6293 2750 50  0000 C CNN
 F 1 "22k" V 6384 2750 50  0000 C CNN
-F 2 "" V 6430 2750 50  0001 C CNN
+F 2 "Resistor_SMD:R_0402_1005Metric" V 6430 2750 50  0001 C CNN
 F 3 "~" H 6500 2750 50  0001 C CNN
 	1    6500 2750
@@
 	6650 2750 6800 2750
 $Comp
-L Digital~Voltmeter:MAN6960 U4
+L Digital_Voltmeter:MAN6960 U4
 U 1 1 5BCE4A3D
 P 7850 2600
@@
 	7500 2750 7500 2650
 $Comp
-L Digital~Voltmeter:ICL7107 U3
+L Digital_Voltmeter:ICL7107 U3
 U 1 1 5BD07790
 P 6800 3400
@@
 $EndComp
 $Comp
-L Digital~Voltmeter:MAN6960 U5
+L Digital_Voltmeter:MAN6960 U5
 U 1 1 5BD08FBF
 P 7850 3650
@@
 F 0 "R6" V 7500 3850 50  0000 C CNN
 F 1 "560" V 7500 4000 50  0000 C CNN
-F 2 "" V 7330 4000 50  0001 C CNN
+F 2 "Resistor_SMD:R_0201_0603Metric" V 7330 4000 50  0001 C CNN
 F 3 "~" H 7400 4000 50  0001 C CNN
 	1    7400 4000
@@
 $EndComp
 $Comp
-L Digital~Voltmeter:MAN6960 U7
+L Digital_Voltmeter:MAN6960 U7
 U 1 1 5BD0C170
 P 7850 5500
@@
 $EndComp
 $Comp
-L Digital~Voltmeter:MAN6960 U6
+L Digital_Voltmeter:MAN6960 U6
 U 1 1 5BD10FF0
 P 7850 4700
@@
 Wire Wire Line
 	8850 5500 8600 5500
-Connection ~ 6800 2750
 Wire Wire Line
 	8600 4700 8850 4700
@@
 Wire Wire Line
 	8850 2600 8850 3650
-Wire Wire Line
-	3400 1900 6800 1900
-Connection ~ 3400 1900
 Connection ~ 6800 1900
 Wire Wire Line
@@
 Wire Wire Line
 	6800 6000 6800 5950
+Wire Wire Line
+	2150 1900 6800 1900
 $EndSCHEMATC

Commit message: working on pcb
Parts:
- added J?: Conn_01x02_Female, symbol Connector:Conn_01x02_Female
- RV1: footprint (none) -> Digital_Voltmeter_Parts:T93YB_TrimPot
- U2: footprint (none) -> ICL7660SIBAZT:SOIC127P600X175-8N
- U3: footprint (none) -> Digital_Voltmeter_Parts:ICL7107CPL&plus_
- U4, U5, U6, U7: footprint (none) -> Digital_Voltmeter_Parts:SC56-11SRWA
Changed lines of the file:
@@
 EESchema Schematic File Version 4
+LIBS:Digital Voltmeter-cache
 EELAYER 26 0
 EELAYER END
@@
 F 0 "U2" H 3200 2650 50  0000 L CNN
 F 1 "ICL7660S" H 3250 2400 50  0000 L CNN
-F 2 "" H 3400 2300 50  0001 C CNN
+F 2 "ICL7660SIBAZT:SOIC127P600X175-8N" H 3400 2300 50  0001 C CNN
 F 3 "" H 3400 2300 50  0001 C CNN
 	1    3400 2300
@@
 Wire Wire Line
 	1550 1900 1150 1900
-Text Label 1350 1900 0    50   ~ 0
+Text Label 1150 1900 0    50   ~ 0
 Vin=9V
 Text Label 2150 1900 0    50   ~ 0
 5V
-Text Label 3750 2300 0    50   ~ 0
--5V
 Wire Wire Line
 	3400 2700 3400 2800
@@
 	2150 2050 2150 2000
 Connection ~ 2150 2000
-Connection ~ 2150 1900
 $Comp
 L Regulator_Linear:L78L05_SO8 U1
@@
 F 0 "RV1" H 5780 2996 50  0000 R CNN
 F 1 "20k" H 5780 2905 50  0000 R CNN
-F 2 "" H 5850 2950 50  0001 C CNN
+F 2 "Digital_Voltmeter_Parts:T93YB_TrimPot" H 5850 2950 50  0001 C CNN
 F 3 "~" H 5850 2950 50  0001 C CNN
 	1    5850 2950
@@
 F 0 "U4" V 8415 2835 50  0000 C CNN
 F 1 "MAN6960" V 8324 2835 50  0000 C CNN
-F 2 "" H 7800 2600 50  0001 C CNN
+F 2 "Digital_Voltmeter_Parts:SC56-11SRWA" H 7800 2600 50  0001 C CNN
 F 3 "" H 7800 2600 50  0001 C CNN
 	1    7850 2600
@@
 Wire Wire Line
 	7500 2750 7500 2650
-$Comp
-L Digital_Voltmeter:ICL7107 U3
-U 1 1 5BD07790
-P 6800 3400
-F 0 "U3" H 6800 4228 50  0000 C CNN
-F 1 "ICL7107" H 6800 4137 50  0000 C CNN
-F 2 "" H 6800 3400 50  0001 C CNN
-F 3 "" H 6800 3400 50  0001 C CNN
-	1    6800 3400
-	1    0    0    -1
-$EndComp
 $Comp
 L Digital_Voltmeter:MAN6960 U5
@@
 F 0 "U5" V 8415 3885 50  0000 C CNN
 F 1 "MAN6960" V 8324 3885 50  0000 C CNN
-F 2 "" H 7800 3650 50  0001 C CNN
+F 2 "Digital_Voltmeter_Parts:SC56-11SRWA" H 7800 3650 50  0001 C CNN
 F 3 "" H 7800 3650 50  0001 C CNN
 	1    7850 3650
@@
 U 1 1 5BD0A81F
 P 7400 4000
-F 0 "R6" V 7500 3850 50  0000 C CNN
+F 0 "R6" V 7400 4000 50  0000 C CNN
 F 1 "560" V 7500 4000 50  0000 C CNN
 F 2 "Resistor_SMD:R_0201_0603Metric" V 7330 4000 50  0001 C CNN
@@
 F 0 "U7" V 8415 5735 50  0000 C CNN
 F 1 "MAN6960" V 8324 5735 50  0000 C CNN
-F 2 "" H 7800 5500 50  0001 C CNN
+F 2 "Digital_Voltmeter_Parts:SC56-11SRWA" H 7800 5500 50  0001 C CNN
 F 3 "" H 7800 5500 50  0001 C CNN
 	1    7850 5500
@@
 F 0 "U6" V 8415 4935 50  0000 C CNN
 F 1 "MAN6960" V 8324 4935 50  0000 C CNN
-F 2 "" H 7800 4700 50  0001 C CNN
+F 2 "Digital_Voltmeter_Parts:SC56-11SRWA" H 7800 4700 50  0001 C CNN
 F 3 "" H 7800 4700 50  0001 C CNN
 	1    7850 4700
@@
 $EndComp
 Wire Wire Line
-	7550 4000 7600 4000
-Wire Wire Line
-	7550 4000 7550 4050
-Connection ~ 7550 4000
+	7250 4000 7250 4050
 $Comp
 L power:GND #PWR0102
 U 1 1 5BD17463
-P 7550 4050
-F 0 "#PWR0102" H 7550 3800 50  0001 C CNN
-F 1 "GND" H 7555 3877 50  0000 C CNN
-F 2 "" H 7550 4050 50  0001 C CNN
-F 3 "" H 7550 4050 50  0001 C CNN
-	1    7550 4050
+P 7250 4050
+F 0 "#PWR0102" H 7250 3800 50  0001 C CNN
+F 1 "GND" H 7255 3877 50  0000 C CNN
+F 2 "" H 7250 4050 50  0001 C CNN
+F 3 "" H 7250 4050 50  0001 C CNN
+	1    7250 4050
 	1    0    0    -1
 $EndComp
 NoConn ~ 7600 2850
-NoConn ~ 7600 5050
+NoConn ~ 7600 4000
 NoConn ~ 7600 5850
 NoConn ~ 7600 2950
@@
 Vin-
 Wire Wire Line
-	6800 2750 6800 1900
-Wire Wire Line
-	6800 1900 8850 1900
-Wire Wire Line
-	8850 1900 8850 2600
-Wire Wire Line
 	8850 5500 8600 5500
 Wire Wire Line
@@
 Wire Wire Line
 	8600 2600 8850 2600
-Connection ~ 8850 2600
 Wire Wire Line
 	8850 2600 8850 3650
-Connection ~ 6800 1900
-Wire Wire Line
-	6800 6000 4600 6000
-Wire Wire Line
-	4600 6000 4600 2300
-Wire Wire Line
-	4600 2300 4000 2300
-Connection ~ 4000 2300
 Wire Wire Line
 	6800 6000 6800 5950
 Wire Wire Line
-	2150 1900 6800 1900
+	3400 1900 2150 1900
+Connection ~ 2150 1900
+Text GLabel 3400 1900 2    50   Input ~ 0
+5V
+$Comp
+L Digital_Voltmeter:ICL7107 U3
+U 1 1 5BD07790
+P 6800 3400
+F 0 "U3" H 6800 4228 50  0000 C CNN
+F 1 "ICL7107" H 6800 4137 50  0000 C CNN
+F 2 "Digital_Voltmeter_Parts:ICL7107CPL&plus_" H 6800 3400 50  0001 C CNN
+F 3 "" H 6800 3400 50  0001 C CNN
+	1    6800 3400
+	1    0    0    -1
+$EndComp
+Text GLabel 4000 2300 2    50   Input ~ 0
+-5V
+Text GLabel 6800 6000 2    50   Input ~ 0
+-5V
+Text GLabel 8850 2600 2    50   Input ~ 0
+5V
+Wire Wire Line
+	1550 2800 1150 2800
+Connection ~ 1550 2800
+Text Label 1150 2800 0    50   ~ 0
+GND
+Text GLabel 6800 2750 2    50   Input ~ 0
+5V
+Connection ~ 7250 4000
+Wire Wire Line
+	7550 4000 7550 5050
+Wire Wire Line
+	7550 5050 7600 5050
+$Comp
+L Connector:Conn_01x02_Female J?
+U 1 1 5BDA935F
+P 800 2250
+F 0 "J?" H 700 2400 50  0000 L CNN
+F 1 "Conn_01x02_Female" H 350 2050 50  0000 L CNN
+F 2 "" H 800 2250 50  0001 C CNN
+F 3 "~" H 800 2250 50  0001 C CNN
+	1    800  2250
+	-1   0    0    -1
+$EndComp
+Wire Wire Line
+	1000 2250 1150 2250
+Wire Wire Line
+	1150 2250 1150 1900
+Wire Wire Line
+	1000 2350 1150 2350
+Wire Wire Line
+	1150 2350 1150 2800
+Text GLabel 800  2250 0    50   Input ~ 0
+Vin=9V
+Text GLabel 800  2350 0    50   Input ~ 0
+GND
 $EndSCHEMATC

Commit message: before changing some components
Parts:
- removed J?: Conn_01x02_Female, symbol Connector:Conn_01x02_Female
Connections:
- wire segments 90 -> 86
Changed lines of the file:
@@
 Wire Wire Line
 	7550 5050 7600 5050
-$Comp
-L Connector:Conn_01x02_Female J?
-U 1 1 5BDA935F
-P 800 2250
-F 0 "J?" H 700 2400 50  0000 L CNN
-F 1 "Conn_01x02_Female" H 350 2050 50  0000 L CNN
-F 2 "" H 800 2250 50  0001 C CNN
-F 3 "~" H 800 2250 50  0001 C CNN
-	1    800  2250
-	-1   0    0    -1
-$EndComp
-Wire Wire Line
-	1000 2250 1150 2250
-Wire Wire Line
-	1150 2250 1150 1900
-Wire Wire Line
-	1000 2350 1150 2350
-Wire Wire Line
-	1150 2350 1150 2800
-Text GLabel 800  2250 0    50   Input ~ 0
-Vin=9V
-Text GLabel 800  2350 0    50   Input ~ 0
-GND
 $EndSCHEMATC

Commit message: replaced parts
Parts:
- C2, C5: footprint Capacitor_SMD:C_0603_1608Metric -> Capacitor_SMD:C_0603_1608Metric_Pad1.05x0.95mm_HandSolder
- C3, C4, C8: footprint Capacitor_SMD:C_0805_2012Metric -> Capacitor_SMD:C_0603_1608Metric_Pad1.05x0.95mm_HandSolder
- C6, C7, C9: footprint Capacitor_SMD:C_0402_1005Metric -> Capacitor_SMD:C_0603_1608Metric_Pad1.05x0.95mm_HandSolder
- R1: footprint Resistor_SMD:R_0805_2012Metric -> Resistor_SMD:R_0603_1608Metric_Pad1.05x0.95mm_HandSolder
- R2, R4, R5: footprint Resistor_SMD:R_0402_1005Metric -> Resistor_SMD:R_0603_1608Metric_Pad1.05x0.95mm_HandSolder
- R3, R6: footprint Resistor_SMD:R_0201_0603Metric -> Resistor_SMD:R_0603_1608Metric_Pad1.05x0.95mm_HandSolder
Changed lines of the file:
@@
 F 0 "C2" H 2328 2346 50  0000 L CNN
 F 1 "2.2u" H 2328 2255 50  0000 L CNN
-F 2 "Capacitor_SMD:C_0603_1608Metric" H 2150 2300 50  0001 C CNN
+F 2 "Capacitor_SMD:C_0603_1608Metric_Pad1.05x0.95mm_HandSolder" H 2150 2300 50  0001 C CNN
 F 3 "" H 2150 2300 50  0001 C CNN
 	1    2150 2300
@@
 F 0 "C3" H 2978 2346 50  0000 L CNN
 F 1 "10u" H 2978 2255 50  0000 L CNN
-F 2 "Capacitor_SMD:C_0805_2012Metric" H 2800 2300 50  0001 C CNN
+F 2 "Capacitor_SMD:C_0603_1608Metric_Pad1.05x0.95mm_HandSolder" H 2800 2300 50  0001 C CNN
 F 3 "" H 2800 2300 50  0001 C CNN
 	1    2800 2300
@@
 F 0 "C4" H 4178 2596 50  0000 L CNN
 F 1 "10u" H 4178 2505 50  0000 L CNN
-F 2 "Capacitor_SMD:C_0805_2012Metric" H 4000 2550 50  0001 C CNN
+F 2 "Capacitor_SMD:C_0603_1608Metric_Pad1.05x0.95mm_HandSolder" H 4000 2550 50  0001 C CNN
 F 3 "" H 4000 2550 50  0001 C CNN
 	1    4000 2550
@@
 F 0 "C6" H 6028 4996 50  0000 L CNN
 F 1 "100nF" H 6028 4905 50  0000 L CNN
-F 2 "Capacitor_SMD:C_0402_1005Metric" H 5850 4950 50  0001 C CNN
+F 2 "Capacitor_SMD:C_0603_1608Metric_Pad1.05x0.95mm_HandSolder" H 5850 4950 50  0001 C CNN
 F 3 "" H 5850 4950 50  0001 C CNN
 	1    5850 4950
@@
 F 0 "C5" H 6028 3696 50  0000 L CNN
 F 1 "10nF" H 6028 3605 50  0000 L CNN
-F 2 "Capacitor_SMD:C_0603_1608Metric" H 5850 3650 50  0001 C CNN
+F 2 "Capacitor_SMD:C_0603_1608Metric_Pad1.05x0.95mm_HandSolder" H 5850 3650 50  0001 C CNN
 F 3 "" H 5850 3650 50  0001 C CNN
 	1    5850 3650
@@
 F 0 "C9" V 6000 5300 50  0000 C CNN
 F 1 "100pF" V 6000 5600 50  0000 C CNN
-F 2 "Capacitor_SMD:C_0402_1005Metric" H 6100 5400 50  0001 C CNN
+F 2 "Capacitor_SMD:C_0603_1608Metric_Pad1.05x0.95mm_HandSolder" H 6100 5400 50  0001 C CNN
 F 3 "" H 6100 5400 50  0001 C CNN
 	1    6100 5400
@@
 F 0 "C8" V 6150 4400 50  0000 C CNN
 F 1 "220nF" V 6150 4700 50  0000 C CNN
-F 2 "Capacitor_SMD:C_0805_2012Metric" H 6100 4500 50  0001 C CNN
+F 2 "Capacitor_SMD:C_0603_1608Metric_Pad1.05x0.95mm_HandSolder" H 6100 4500 50  0001 C CNN
 F 3 "" H 6100 4500 50  0001 C CNN
 	1    6100 4500
@@
 F 0 "C7" V 6150 4000 50  0000 C CNN
 F 1 "47nF" V 6150 4250 50  0000 C CNN
-F 2 "Capacitor_SMD:C_0402_1005Metric" H 6100 4100 50  0001 C CNN
+F 2 "Capacitor_SMD:C_0603_1608Metric_Pad1.05x0.95mm_HandSolder" H 6100 4100 50  0001 C CNN
 F 3 "" H 6100 4100 50  0001 C CNN
 	1    6100 4100
@@
 F 0 "R4" V 6150 5450 50  0000 C CNN
 F 1 "180k" V 6150 5800 50  0000 C CNN
-F 2 "Resistor_SMD:R_0402_1005Metric" V 6030 5600 50  0001 C CNN
+F 2 "Resistor_SMD:R_0603_1608Metric_Pad1.05x0.95mm_HandSolder" V 6030 5600 50  0001 C CNN
 F 3 "~" H 6100 5600 50  0001 C CNN
 	1    6100 5600
@@
 F 0 "R3" V 6150 4150 50  0000 C CNN
 F 1 "470k" V 6150 4500 50  0000 C CNN
-F 2 "Resistor_SMD:R_0201_0603Metric" V 6030 4300 50  0001 C CNN
+F 2 "Resistor_SMD:R_0603_1608Metric_Pad1.05x0.95mm_HandSolder" V 6030 4300 50  0001 C CNN
 F 3 "~" H 6100 4300 50  0001 C CNN
 	1    6100 4300
@@
 F 0 "R2" H 5570 3696 50  0000 L CNN
 F 1 "12k" H 5570 3605 50  0000 L CNN
-F 2 "Resistor_SMD:R_0402_1005Metric" V 5430 3650 50  0001 C CNN
+F 2 "Resistor_SMD:R_0603_1608Metric_Pad1.05x0.95mm_HandSolder" V 5430 3650 50  0001 C CNN
 F 3 "~" H 5500 3650 50  0001 C CNN
 	1    5500 3650
@@
 F 0 "R1" V 4943 3900 50  0000 C CNN
 F 1 "1M" V 5034 3900 50  0000 C CNN
-F 2 "Resistor_SMD:R_0805_2012Metric" V 5080 3900 50  0001 C CNN
+F 2 "Resistor_SMD:R_0603_1608Metric_Pad1.05x0.95mm_HandSolder" V 5080 3900 50  0001 C CNN
 F 3 "~" H 5150 3900 50  0001 C CNN
 	1    5150 3900
@@
 F 0 "R5" V 6293 2750 50  0000 C CNN
 F 1 "22k" V 6384 2750 50  0000 C CNN
-F 2 "Resistor_SMD:R_0402_1005Metric" V 6430 2750 50  0001 C CNN
+F 2 "Resistor_SMD:R_0603_1608Metric_Pad1.05x0.95mm_HandSolder" V 6430 2750 50  0001 C CNN
 F 3 "~" H 6500 2750 50  0001 C CNN
 	1    6500 2750
@@
 F 0 "R6" V 7400 4000 50  0000 C CNN
 F 1 "560" V 7500 4000 50  0000 C CNN
-F 2 "Resistor_SMD:R_0201_0603Metric" V 7330 4000 50  0001 C CNN
+F 2 "Resistor_SMD:R_0603_1608Metric_Pad1.05x0.95mm_HandSolder" V 7330 4000 50  0001 C CNN
 F 3 "~" H 7400 4000 50  0001 C CNN
 	1    7400 4000

Commit message: passing DMC
Parts:
- added J1, J2: Conn_01x02_Male, Connector_PinHeader_2.54mm:PinHeader_1x02_P2.54mm_Vertical, symbol Connector:Conn_01x02_Male
Connections:
- wire segments 86 -> 90
Changed lines of the file:
@@
 	2800 2550 3050 2550
 Wire Wire Line
-	1550 1900 1150 1900
-Text Label 1150 1900 0    50   ~ 0
+	1550 1900 1200 1900
+Text Label 1200 1900 0    50   ~ 0
 Vin=9V
 Text Label 2150 1900 0    50   ~ 0
@@
 Text GLabel 8850 2600 2    50   Input ~ 0
 5V
-Wire Wire Line
-	1550 2800 1150 2800
-Connection ~ 1550 2800
-Text Label 1150 2800 0    50   ~ 0
-GND
 Text GLabel 6800 2750 2    50   Input ~ 0
 5V
@@
 Wire Wire Line
 	7550 5050 7600 5050
+$Comp
+L Connector:Conn_01x02_Male J1
+U 1 1 5BDA9824
+P 4650 3650
+F 0 "J1" H 4622 3530 50  0000 R CNN
+F 1 "Conn_01x02_Male" H 4622 3621 50  0000 R CNN
+F 2 "Connector_PinHeader_2.54mm:PinHeader_1x02_P2.54mm_Vertical" H 4650 3650 50  0001 C CNN
+F 3 "~" H 4650 3650 50  0001 C CNN
+	1    4650 3650
+	1    0    0    1
+$EndComp
+Wire Wire Line
+	4850 3550 4850 3400
+Wire Wire Line
+	4850 3650 4850 3900
+$Comp
+L Connector:Conn_01x02_Male J2
+U 1 1 5BDB28C4
+P 1000 2250
+F 0 "J2" H 1106 2428 50  0000 C CNN
+F 1 "Conn_01x02_Male" H 1106 2337 50  0000 C CNN
+F 2 "Connector_PinHeader_2.54mm:PinHeader_1x02_P2.54mm_Vertical" H 1000 2250 50  0001 C CNN
+F 3 "~" H 1000 2250 50  0001 C CNN
+	1    1000 2250
+	1    0    0    -1
+$EndComp
+Wire Wire Line
+	1200 2350 1200 2800
+Wire Wire Line
+	1200 2800 1550 2800
+Connection ~ 1550 2800
+Wire Wire Line
+	1200 2250 1200 1900
 $EndSCHEMATC
